File: Hardware/jade_hardware.sch (KiCad schematic (older format))
At the start: 37 parts, among them J1 PJ302M, J2 PJ302M, J3 PJ302M, J4 PJ302M, J5 Conn_02x05_Odd_Even, J6 Conn_02x03_Odd_Even, J7 PJ302M, J8 PJ302M, Q1 MMBT3904, Q2 MMBT3904, Q3 MMBT3904, Q4 MMBT3904, U1 SeeeduinoXIAO, U2 LM358

Commit message: Eurorack main board Rev.B
Parts:
- removed R10: 10k, Resistor_SMD:R_0603_1608Metric_Pad0.98x0.95mm_HandSolder, symbol Device:R_Small
- added R11: 47k, Resistor_SMD:R_0603_1608Metric_Pad0.98x0.95mm_HandSolder, symbol Device:R_Small
- R12: value 10k -> 47k
- renumbered R11 to R10
Connections:
- net CLOCK_OUT: now also U2.3 (+), R11.2; no longer R12.2
- net GATE_OUT: now also R12.2, U2.5 (+)
- net GND: now also R12.1, R11.1
Other:
- moved on the sheet: C2, J7, R13, R15, R9, U2B, U2C

Commit message: Schematic Rev.C
Parts:
- removed J8: PJ302M, Akiyuki_Footprint:PJ302M, symbol Akiyuki_Connector:PJ302M
- removed Q1, Q2, Q3, Q4: MMBT3904, Package_TO_SOT_SMD:SOT-23, symbol Transistor_BJT:MMBT3904
- removed R10, R9: 39k, Resistor_SMD:R_0603_1608Metric_Pad0.98x0.95mm_HandSolder, symbol Device:R_Small
- removed R11, R12: 47k, Resistor_SMD:R_0603_1608Metric_Pad0.98x0.95mm_HandSolder, symbol Device:R_Small
- removed R13, R14: 56k, Resistor_SMD:R_0603_1608Metric_Pad0.98x0.95mm_HandSolder, symbol Device:R_Small
- removed R15, R16: 1k, Resistor_SMD:R_0603_1608Metric_Pad0.98x0.95mm_HandSolder, symbol Device:R_Small
- removed R3: 100k, Resistor_SMD:R_0603_1608Metric_Pad0.98x0.95mm_HandSolder, symbol Device:R_Small
- removed U2: LM358, Package_SO:SOP-8_3.9x4.9mm_P1.27mm, symbol Amplifier_Operational:LM358
- added C3, C4: 0.1u, Capacitor_SMD:C_0402_1005Metric_Pad0.74x0.62mm_HandSolder, symbol Device:C_Small
- added J6: PJ302M, Akiyuki_Footprint:PJ302M, symbol Akiyuki_Connector:PJ302M
- added R7: 2k2, Resistor_SMD:R_0402_1005Metric_Pad0.72x0.64mm_HandSolder, symbol Device:R_Small
- added SW1: SW_DIP_x02, Akiyuki_Footprint:OTAX_KHS_2, symbol Switch:SW_DIP_x02
- added U1: TLP293-4, Package_SO:SOIC-16_4.55x10.3mm_P1.27mm, symbol Isolator:TLP291-4
- added U3: MIC39100, Package_TO_SOT_SMD:SOT-223-3_TabPin2, symbol Akiyuki_IC:MIC39100
- added U4, U5: TLP291, Package_SO:SOIC-4_4.55x2.6mm_P1.27mm, symbol Isolator:TLP291
- added U6: ADuM1250, Package_SO:SOIC-8_3.9x4.9mm_P1.27mm, symbol Akiyuki_IC:ADuM1250
- C2: value 0.1u -> 10u; footprint Capacitor_SMD:C_0603_1608Metric_Pad1.08x0.95mm_HandSolder -> Capacitor_SMD:C_0805_2012Metric_Pad1.18x1.45mm_HandSolder
- J8: renamed from J6; value Conn_02x03_Odd_Even -> monome ii
- R1, R2, R4: footprint Resistor_SMD:R_0603_1608Metric_Pad0.98x0.95mm_HandSolder -> Resistor_SMD:R_0402_1005Metric_Pad0.72x0.64mm_HandSolder
- R3: renamed from R7; footprint Resistor_SMD:R_0603_1608Metric_Pad0.98x0.95mm_HandSolder -> Resistor_SMD:R_0402_1005Metric_Pad0.72x0.64mm_HandSolder
- R5, R6: value 100k -> 47k; footprint Resistor_SMD:R_0603_1608Metric_Pad0.98x0.95mm_HandSolder -> Resistor_SMD:R_0402_1005Metric_Pad0.72x0.64mm_HandSolder
- R8: value 100k -> 2k2; footprint Resistor_SMD:R_0603_1608Metric_Pad0.98x0.95mm_HandSolder -> Resistor_SMD:R_0402_1005Metric_Pad0.72x0.64mm_HandSolder
- renumbered U1 to U2
Connections:
- net +12V: now also R5.2, R6.2, U3.1 (VI); no longer C2.1
- net CLOCK_OUT: now also U4.1
- net GATE_IN1: now also U1.16
- net GATE_IN2: now also U1.14
- net GATE_IN3: now also U1.12
- net GATE_IN4: now also U1.10
- net GATE_OUT: now also U5.1
- net SCL: now also U6.3 (SCL1); no longer J8.3 (Pin_3), J8.4 (Pin_4)
- net SDA: now also U6.2 (SDA1); no longer J8.1 (Pin_1), J8.2 (Pin_2)
- net +3V3: now reaches U2.12 (3V3)
- net +3V3: now also C3.1, U6.1 (VDD1)
- net at J1.3, R1.2: now also D1.1 (K), U1.1
- net at J2.3, R2.2: now also D2.1 (K), U1.3
- net at J3.3: now also D3.1 (K), R3.2, U1.5
- net at J4.3, R4.2: now also D4.1 (K), U1.7
- net at J7.3: now also R6.1, U5.4
- net GND renamed GNDA
- net GNDA: now also R1.1, R2.1, R4.1, C4.1, J6.1, J6.2, U1.2, U1.4, U1.6, U1.8, U3.2 (GND), U4.3, U5.3, U6.5 (GND2); no longer R5.1, R6.1, R8.1, U2.13 (GND)
- new net: J8.1 (Pin_1), J8.2 (Pin_2), SW1.3, U6.7 (SDA2)
- new net: J8.3 (Pin_3), J8.4 (Pin_4), SW1.4, U6.6 (SCL2)
- new net: J6.3, R5.1, U4.4
- new net: R7.2, SW1.2
- new net: R8.2, SW1.1
- new net +3.3VA: C2.1, C4.2, R7.1, R8.1, U3.3 (VO), U6.8 (VDD2)
- new net GNDD: C3.2, U1.11, U1.13, U1.15, U1.9, U2.13 (GND), U4.2, U5.2, U6.4 (GND1)
- no-connect marks 7 -> 6
Other:
- note added: "Enanble I2C pullup"
- note added: "Gate output"
- note added: "When the input impedance to receive this CV/Gate is 100kΩ, \nthe voltage drops to about 8V."
- note removed: "0V to 8V\n"
- moved on the sheet: D3, J3, J7, J8, R3, U2A, U2B
