File: Hardware/jade_hardware.kicad_pcb (KiCad board)
At the start: 2 copper layers, 30 x 110 mm, 37 parts, among them J1 PJ302M, J2 PJ302M, J3 PJ302M, J4 PJ302M, J5 Conn_02x05_Odd_Even, J6 Conn_02x03_Odd_Even, J7 PJ302M, J8 PJ302M, Q1 MMBT3904, Q2 MMBT3904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

Commit message: Eurorack main board Rev.B
Parts:
- removed the R10 at (143.0, 136.0)
- added R11: 47k, Resistor_SMD:R_0603_1608Metric_Pad0.98x0.95mm_HandSolder, F.Cu at (138.7, 132.6)
- D1, D2, D3, D4: value 1N4148 -> 1N4148W
- D5: value 1N5819 -> 1N5819HW
- R12: value 10k -> 47k
- moved R12 6.83 mm to (140.5, 142.9), turned to 90 degrees
- moved D3 4.60 mm to (136.5, 92.4)
- moved R3 4.60 mm to (133.0, 93.1)
- moved R7 4.60 mm to (134.5, 93.1)
- moved Q4 2.77 mm to (119.5, 135.5), turned to 270 degrees
- moved Q3 2.65 mm to (124.9, 135.5), turned to 270 degrees
- renumbered R11 to R10
Connections:
- R12 pad 1: Net-(R12-Pad1) -> GND
- R12 pad 2: /CLOCK_OUT -> /GATE_OUT
- U2 pad 3: Net-(R12-Pad1) -> /CLOCK_OUT
- U2 pad 5: Net-(R10-Pad1) (its old number) -> /GATE_OUT
Routing:
- net /GATE_OUT: track 28.3 -> 45.8 mm
- net Net-(R10-Pad1) (its old number): track 15.0 -> 0.00 mm
- net /CLOCK_OUT: track 28.5 -> 39.0 mm
- net Net-(R12-Pad1): track 9.52 -> 0.00 mm
- net Net-(D3-Pad1): track 52.5 -> 47.0 mm
- net Net-(J3-Pad3): track 6.80 -> 10.6 mm
- net /GATE_IN4: track 6.96 -> 8.88 mm
- net /GATE_IN3: track 5.19 -> 6.29 mm
- net Net-(D4-Pad1): track 33.0 -> 32.0 mm
- net GND: vias 29 -> 38
Other:
- board text added: "Akiyuki Okayasu"
- board text added: "JLCJLCJLCJLC"
- board text added: "Rev. B"
- board text removed: "Rev. A"

Commit message: update all changes before stash
Parts:
- removed Q1, Q2, Q3, Q4: MMBT3904, Package_TO_SOT_SMD:SOT-23
- removed R10, R9: 39k, Resistor_SMD:R_0603_1608Metric_Pad0.98x0.95mm_HandSolder
- removed R11, R12: 47k, Resistor_SMD:R_0603_1608Metric_Pad0.98x0.95mm_HandSolder
- removed R13, R14: 56k, Resistor_SMD:R_0603_1608Metric_Pad0.98x0.95mm_HandSolder
- removed R15, R16: 1k, Resistor_SMD:R_0603_1608Metric_Pad0.98x0.95mm_HandSolder
- added C3: 0.1u, Capacitor_SMD:C_0402_1005Metric_Pad0.74x0.62mm_HandSolder, F.Cu at (169.8, 92.4)
- added C4: 0.1u, Capacitor_SMD:C_0402_1005Metric_Pad0.74x0.62mm_HandSolder, F.Cu at (184.6, 92.4)
- added SW1: SW_DIP_x02, Akiyuki_Footprint:OTAX_KHS_2, F.Cu at (175.0, 66.5)
- added U3: MIC39100, Package_TO_SOT_SMD:SOT-223-3_TabPin2, F.Cu at (159.0, 88.5)
- added U4: TLP291, Package_SO:SOIC-4_4.55x2.6mm_P1.27mm, B.Cu at (119.0, 137.5)
- added U5: TLP291, Package_SO:SOIC-4_4.55x2.6mm_P1.27mm, B.Cu at (123.5, 137.5)
- added U6: ADuM1250, Package_SO:SOIC-8_3.9x4.9mm_P1.27mm, F.Cu at (151.0, 132.0)
- C2: value 0.1u -> 10u; footprint Capacitor_SMD:C_0603_1608Metric_Pad1.08x0.95mm_HandSolder -> Capacitor_SMD:C_0805_2012Metric_Pad1.18x1.45mm_HandSolder
- J6: value Conn_02x03_Odd_Even -> PJ302M; footprint Connector_PinHeader_2.54mm:PinHeader_2x03_P2.54mm_Horizontal -> Akiyuki_Footprint:PJ302M
- J8: value PJ302M -> monome ii; footprint Akiyuki_Footprint:PJ302M -> Connector_PinHeader_2.54mm:PinHeader_2x03_P2.54mm_Horizontal
- R1, R2, R3, R4: footprint Resistor_SMD:R_0603_1608Metric_Pad0.98x0.95mm_HandSolder -> Resistor_SMD:R_0402_1005Metric_Pad0.72x0.64mm_HandSolder
- R5, R6: value 100k -> 47k; footprint Resistor_SMD:R_0603_1608Metric_Pad0.98x0.95mm_HandSolder -> Resistor_SMD:R_0402_1005Metric_Pad0.72x0.64mm_HandSolder
- R7, R8: value 100k -> 2k2; footprint Resistor_SMD:R_0603_1608Metric_Pad0.98x0.95mm_HandSolder -> Resistor_SMD:R_0402_1005Metric_Pad0.72x0.64mm_HandSolder
- U1: value SeeeduinoXIAO -> TLP293-4; footprint Akiyuki_Footprint:Seeeduino_XIAO_NonBottomPad -> Package_SO:SOIC-16_4.55x10.3mm_P1.27mm
- U2: value LM358 -> SeeeduinoXIAO; footprint Package_SO:SOP-8_3.9x4.9mm_P1.27mm -> Akiyuki_Footprint:Seeeduino_XIAO_NonBottomPad
- moved U1 37.6 mm to (138.0, 120.5), turned to 0 degrees
- moved U2 34.2 mm to (136.0, 157.5)
- moved J6 32.4 mm to (115.0, 130.0)
- moved J8 32.3 mm to (135.5, 102.5)
- moved R6 19.4 mm to (153.7, 79.5)
- moved R5 18.7 mm to (154.2, 74.0)
- moved C2 17.0 mm to (153.0, 117.5)
- moved D1 4.27 mm to (133.5, 73.5), turned to 270 degrees
- moved R2 3.20 mm to (135.5, 80.0)
- moved D2 3.01 mm to (133.5, 81.0), turned to 270 degrees
- moved R1 2.50 mm to (135.5, 72.5)
Connections:
- C1 pad 2: GND -> GNDA
- C2 pad 1: +12V -> +3.3VA
- C2 pad 2: GND -> GNDA
- D1 pad 2: GND -> GNDA
- D2 pad 2: GND -> GNDA
- D3 pad 2: GND -> GNDA
- D4 pad 2: GND -> GNDA
- J1 pad 1: GND -> GNDA
- J1 pad 2: GND -> GNDA
- J1 pad 3: Net-(J1-Pad3) -> Net-(D1-Pad1)
- J2 pad 1: GND -> GNDA
- J2 pad 2: GND -> GNDA
- J2 pad 3: Net-(J2-Pad3) -> Net-(D2-Pad1)
- J3 pad 1: GND -> GNDA
- J3 pad 2: GND -> GNDA
- J3 pad 3: Net-(J3-Pad3) -> Net-(D3-Pad1)
- J4 pad 1: GND -> GNDA
- J4 pad 2: GND -> GNDA
- J4 pad 3: Net-(J4-Pad3) -> Net-(D4-Pad1)
- J5 pad 10: Net-(J5-Pad10) -> (no net)
- J5 pad 3: GND -> GNDA
- J5 pad 4: GND -> GNDA
- J5 pad 5: GND -> GNDA
- J5 pad 6: GND -> GNDA
- J5 pad 7: GND -> GNDA
- J5 pad 8: GND -> GNDA
- J5 pad 9: Net-(J5-Pad9) -> (no net)
- J6 pad 1: /SDA -> GNDA
- J6 pad 2: /SDA -> GNDA
- J6 pad 3: /SCL -> Net-(J6-Pad3)
- J7 pad 1: GND -> GNDA
- J7 pad 2: GND -> GNDA
- J8 pad 1: GND -> Net-(J8-Pad1)
- J8 pad 2: GND -> Net-(J8-Pad1)
- R1 pad 1: Net-(D1-Pad1) -> GNDA
- R1 pad 2: Net-(J1-Pad3) -> Net-(D1-Pad1)
- R2 pad 1: Net-(D2-Pad1) -> GNDA
- R2 pad 2: Net-(J2-Pad3) -> Net-(D2-Pad1)
- R3 pad 1: Net-(D3-Pad1) -> GNDA
- R3 pad 2: Net-(J3-Pad3) -> Net-(D3-Pad1)
- R4 pad 1: Net-(D4-Pad1) -> GNDA
- R4 pad 2: Net-(J4-Pad3) -> Net-(D4-Pad1)
- R5 pad 1: GND -> Net-(J6-Pad3)
- R5 pad 2: Net-(D1-Pad1) -> +12V
- R6 pad 1: GND -> Net-(J7-Pad3)
- R6 pad 2: Net-(D2-Pad1) -> +12V
- R7 pad 1: GND -> +3.3VA
- R7 pad 2: Net-(D3-Pad1) -> Net-(R7-Pad2)
- R8 pad 1: GND -> +3.3VA
- R8 pad 2: Net-(D4-Pad1) -> Net-(R8-Pad2)
- U1 pad 1: Net-(U1-Pad1) -> Net-(D1-Pad1)
- U1 pad 10: /GATE_IN3 -> /GATE_IN4
- U1 pad 11: /GATE_IN4 -> GNDD
- U1 pad 12: Net-(U1-Pad12) -> /GATE_IN3
- U1 pad 13: GND -> GNDD
- U1 pad 14: Net-(U1-Pad14) -> /GATE_IN2
- U1 pad 2: Net-(U1-Pad2) -> GNDA
- U1 pad 3: /CLOCK_OUT -> Net-(D2-Pad1)
- U1 pad 4: /GATE_OUT -> GNDA
- U1 pad 5: /SDA -> Net-(D3-Pad1)
- U1 pad 6: /SCL -> GNDA
- U1 pad 7: /GATE_IN1 -> Net-(D4-Pad1)
- U1 pad 8: Net-(U1-Pad8) -> GNDA
- U1 pad 9: /GATE_IN2 -> GNDD
- U2 pad 1: Net-(R14-Pad1) -> (no net)
- U2 pad 2: Net-(R10-Pad1) -> (no net)
- U2 pad 4: GND -> /GATE_OUT
- U2 pad 5: /GATE_OUT -> /SDA
- U2 pad 6: Net-(R13-Pad2) -> /SCL
- U2 pad 7: Net-(R13-Pad1) -> /GATE_IN1
- U2 pad 8: +12V -> (no net)
Routing:
- net Net-(D1-Pad1): track 82.9 -> 15.5 mm, vias 2 -> 0
- net /SDA: track 62.8 -> 0.00 mm, vias 1 -> 0
- net /SCL: track 60.1 -> 0.00 mm, vias 1 -> 0
- net +12V: track 49.1 -> 2.35 mm
- net Net-(D2-Pad1): track 56.9 -> 10.5 mm, vias 2 -> 0
- net /GATE_OUT: track 45.8 -> 0.00 mm
- net /CLOCK_OUT: track 39.0 -> 0.00 mm
- net Net-(D3-Pad1): track 47.0 -> 10.6 mm
- net Net-(D4-Pad1): track 32.0 -> 13.6 mm
- net Net-(J1-Pad3): track 17.5 -> 0.00 mm
- net Net-(J4-Pad3): track 13.5 -> 0.00 mm
- net Net-(J2-Pad3): track 12.1 -> 0.00 mm
- net Net-(J3-Pad3): track 10.6 -> 0.00 mm
- net /GATE_IN4: track 8.88 -> 0.00 mm
- net /GATE_IN1: track 8.78 -> 0.00 mm
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- removed copper zone on B.Cu, net GND
- removed copper zone on F.Cu, net GND
